Commit message: upd

File: urdf/razbot2.urdf.xacro (robot description, xacro)
@@ -3,4 +3,6 @@
   <!-- Include wheel macro -->
   <xacro:include filename="$(find razbot2_description)/urdf/wheel.urdf.xacro" />
+  <!-- Include arm macro -->
+  <xacro:include filename="$(find razbot2_description)/urdf/razbot2_arm/razbot2_arm.urdf.xacro"/>
   <!-- <property> tags encode important robot paremeters. It's helpful to break
   these out from the rest of the description for easy manipulation -->
@@ -42,5 +44,5 @@
       <origin xyz="0 0 0" rpy="0 0 0" />
       <geometry>
-        <mesh filename="package://razbot2_description/meshes/base.stl" />
+        <mesh filename="package://razbot2_description/meshes/razbot2_base/base.stl" />
       </geometry>
       <material name="Blue" />
@@ -84,3 +86,7 @@
     <origin xyz="${-wheel_base/2} ${-wheel_track/2} ${wheel_vertical_offset}" rpy="0 0 0" />
   </xacro:razbot2_wheel>
+  <!-- Add the razbot2 arm onto the platform -->
+  <xacro:razbot2_arm arm_prefix="">
+    <origin xyz="0 0 0" rpy="0 0 0"/>
+  </xacro:razbot2_arm>
 </robot>

Commit message: Added non tested arm

File: urdf/razbot2.urdf.xacro (robot description, xacro)
@@ -86,6 +86,20 @@
     <origin xyz="${-wheel_base/2} ${-wheel_track/2} ${wheel_vertical_offset}" rpy="0 0 0" />
   </xacro:razbot2_wheel>
+  <link name="razbot2_mounting_plate">
+     <visual>
+      <origin xyz="0 0 0" rpy="0 0 0" />
+      <geometry>
+        <box size="1.15 18.5 0.05"/>
+      </geometry>
+    </visual>
+    <collision>
+      <origin xyz="0 0 0" rpy="0 0 0" />
+      <geometry>
+         <box size="1.15 18.5 0.05"/>
+      </geometry>
+    </collision>
+  </link>
   <!-- Add the razbot2 arm onto the platform -->
-  <xacro:razbot2_arm arm_prefix="">
+  <xacro:razbot2_arm arm_prefix="" mounting_link="razbot2_mounting_plate">
     <origin xyz="0 0 0" rpy="0 0 0"/>
   </xacro:razbot2_arm>

File: urdf/razbot2_arm/razbot2_arm.urdf.xacro (robot description, xacro)
@@ -1,9 +1,9 @@
 <?xml version="1.0"?>
 <robot name="razbot2_arm" xmlns:xacro="http://ros.org/wiki/xacro">
-  <xacro:macro name="razbot2_arm" params="prefix *origin">
+  <xacro:macro name="razbot2_arm" params="prefix mounting_link *origin">
     <!-- Arm base link and joint to link_0 -->
     <link name="${prefix}razbot2_arm_base_link">
       <visual>
-        <origin xyz="0 0 0" rpy="0 0 0 "/>
+        <xacro:insert_block name="origin"/>
         <geometry>
           <mesh filename="package://razbot2_description/meshes/razbot2_arm/razbot2_arm_base_link.stl" />
@@ -12,5 +12,5 @@
       </visual>
       <collision>
-        <origin xyz="0 0 0" rpy="0 0 0" />
+        <xacro:insert_block name="origin"/>
         <geometry>
           <mesh filename="package://razbot2_description/meshes/razbot2_arm/razbot2_arm_base_link.stl" />
@@ -32,4 +32,9 @@
       <material>Gazebo/Grey</material>
     </gazebo>
+    <joint name="${prefix}razbot2_arm_mounting_joint" type="revolute">
+      <parent link="${mounting_link}"/>
+      <child link="${prefix}razbot2_arm_base_link"/>
+      <axis xyz="0 0 0" rpy="0 0 0" />
+    </joint>
     <joint name="${prefix}razbot2_arm_base_link_to_0_joint" type="revolute">
       <parent link="${prefix}razbot2_arm_base_link"/>
@@ -37,4 +42,189 @@
       <axis xyz="0 0 0" rpy="0 0 0" />
     </joint>
+   <!-- razbot2_arm_link_0 -->
+   <link name="${prefix}razbot2_arm_link_0">
+      <visual>
+        <origin xyz="0 0 0" rpy="0 0 0 "/>
+        <geometry>
+          <mesh filename="package://razbot2_description/meshes/razbot2_arm/razbot2_arm_link_0.stl" />
+        </geometry>
+        <material name="Grey" />
+      </visual>
+      <collision>
+        <origin xyz="0 0 0" rpy="0 0 0" />
+        <geometry>
+          <mesh filename="package://razbot2_description/meshes/razbot2_arm/razbot2_arm_link_0.stl" />
+        </geometry>
+      </collision>
+      <inertial>
+        <origin xyz="0 0.1 0"/>
+        <mass value="0.15" />
+        <inertia  ixx="0.0001" ixy="0" ixz="0"
+                  iyy="0.0001" iyz="0"
+                  izz="0.0001" />
+      </inertial>
+    </link>
+    <gazebo reference="${prefix}razbot2_arm_link_0">
+      <mu1 value="200.0"/>
+      <mu2 value="100.0"/>
+      <kp value="10000000.0" />
+      <kd value="1.0" />
+      <material>Gazebo/Grey</material>
+    </gazebo>
+    <joint name="${prefix}razbot2_arm_link_0_to_link_1" type="revolute">
+      <parent link="${prefix}razbot2_arm_link_0"/>
+      <child link="${prefix}razbot2_arm_link_1"/>
+      <axis xyz="0 0 0" rpy="0 0 0" />
+    </joint>
+    <!-- razbot2_arm_link_1 -->
+    <link name="${prefix}razbot2_arm_link_1">
+      <visual>
+        <origin xyz="0 0 0" rpy="0 0 0 "/>
+        <geometry>
+          <mesh filename="package://razbot2_description/meshes/razbot2_arm/razbot2_arm_link_1.stl" />
+        </geometry>
+        <material name="Grey" />
+      </visual>
+      <collision>
+        <origin xyz="0 0 0" rpy="0 0 0" />
+        <geometry>
+          <mesh filename="package://razbot2_description/meshes/razbot2_arm/razbot2_arm_link_1.stl" />
+        </geometry>
+      </collision>
+      <inertial>
+        <origin xyz="0 0.1 0"/>
+        <mass value="0.15" />
+        <inertia  ixx="0.0001" ixy="0" ixz="0"
+                  iyy="0.0001" iyz="0"
+                  izz="0.0001" />
+      </inertial>
+    </link>
+    <gazebo reference="${prefix}razbot2_arm_link-2">
+      <mu1 value="200.0"/>
+      <mu2 value="100.0"/>
+      <kp value="10000000.0" />
+      <kd value="1.0" />
+      <material>Gazebo/Grey</material>
+    </gazebo>
+    <joint name="${prefix}razbot2_arm_link_1_to_link_2" type="revolute">
+      <parent link="${prefix}razbot2_arm_link_1"/>
+      <child link="${prefix}razbot2_arm_link_2"/>
+      <axis xyz="0 0 0" rpy="0 0 0" />
+    </joint>
+   <!-- razbot2_arm_link_3 -->
+   <link name="${prefix}razbot2_arm_link_3">
+      <visual>
+        <origin xyz="0 0 0" rpy="0 0 0 "/>
+        <geometry>
+          <mesh filename="package://razbot2_description/meshes/razbot2_arm/razbot2_arm_link_3.stl" />
+        </geometry>
+        <material name="Grey" />
+      </visual>
+      <collision>
+        <origin xyz="0 0 0" rpy="0 0 0" />
+        <geometry>
+          <mesh filename="package://razbot2_description/meshes/razbot2_arm/razbot2_arm_link_3.stl" />
+        </geometry>
+      </collision>
+      <inertial>
+        <origin xyz="0 0.1 0"/>
+        <mass value="0.15" />
+        <inertia  ixx="0.0001" ixy="0" ixz="0"
+                  iyy="0.0001" iyz="0"
+                  izz="0.0001" />
+      </inertial>
+    </link>
+    <gazebo reference="${prefix}razbot2_arm_link_3">
+      <mu1 value="200.0"/>
+      <mu2 value="100.0"/>
+      <kp value="10000000.0" />
+      <kd value="1.0" />
+      <material>Gazebo/Grey</material>
+    </gazebo>
+    <joint name="${prefix}razbot2_arm_link_1_to_link_2" type="revolute">
+      <parent link="${prefix}razbot2_arm_link_2"/>
+      <child link="${prefix}razbot2_arm_link_3"/>
+      <axis xyz="0 0 0" rpy="0 0 0" />
+    </joint>
+   <!-- Gripper mounting plate -->
+   <link name="${prefix}razbot2_arm_gripper_mounting_plate">
+      <visual>
+        <origin xyz="0 0 0" rpy="0 0 0 "/>
+        <geometry>
+          <mesh filename="package://razbot2_description/meshes/razbot2_arm/razbot2_gripper_mounting_plate.stl" />
+        </geometry>
+        <material name="Grey" />
+      </visual>
+      <collision>
+        <origin xyz="0 0 0" rpy="0 0 0" />
+        <geometry>
+          <mesh filename="package://razbot2_description/meshes/razbot2_arm/razbot2_gripper_mounting_plate.stl" />
+        </geometry>
+      </collision>
+      <inertial>
+        <origin xyz="0 0.1 0"/>
+        <mass value="0.15" />
+        <inertia  ixx="0.0001" ixy="0" ixz="0"
+                  iyy="0.0001" iyz="0"
+                  izz="0.0001" />
+      </inertial>
+    </link>
+    <gazebo reference="${prefix}razbot2_gripper_mounting_plate">
+      <mu1 value="200.0"/>
+      <mu2 value="100.0"/>
+      <kp value="10000000.0" />
+      <kd value="1.0" />
+      <material>Gazebo/Grey</material>
+    </gazebo>
+    <joint name="${prefix}razbot2_arm_to_gripper_plate" type="fixed">
+      <parent link="${prefix}razbot2_arm_link_3"/>
+      <child link="${prefix}razbot2_arm_gripper_mounting_plate"/>
+      <axis xyz="0 0 0" rpy="0 0 0" />
+    </joint>
+    <!-- Left finger gripper -->
+    <xacro:gripper_finger prefix="left">
+       <origin xyz="0 0 0" rpy="0 0 0"/>
+    </xacro:gripper_finger>
+    <!-- Right finger gripper -->
+    <xacro:gripper_finger prefix="right">
+       <origin xyz="0 0 0" rpy="0 0 0"/>
+    </xacro:gripper_finger>
   </xacro:macro>
+  <!-- gripper finger xacro -->
+   <xacro:macro name="gripper_finger" params="prefix *origin">
+      <link name="${prefix}razbot2_gripper_finger">
+      <visual>
+        <xacro:insert_block name="origin"/>
+        <geometry>
+          <mesh filename="package://razbot2_description/meshes/razbot2_arm/razbot2_gripper_finger.stl" />
+        </geometry>
+        <material name="Grey" />
+      </visual>
+      <collision>
+        <xacro:insert_block name="origin"/>
+        <geometry>
+          <mesh filename="package://razbot2_description/meshes/razbot2_arm/razbot2_gripper_finger.stl" />
+        </geometry>
+      </collision>
+      <inertial>
+        <origin xyz="0 0.1 0"/>
+        <mass value="0.15" />
+        <inertia  ixx="0.0001" ixy="0" ixz="0"
+                  iyy="0.0001" iyz="0"
+                  izz="0.0001" />
+      </inertial>
+    </link>
+    <gazebo reference="${prefix}razbot2_gripper_finger">
+      <mu1 value="200.0"/>
+      <mu2 value="100.0"/>
+      <kp value="10000000.0" />
+      <kd value="1.0" />
+      <material>Gazebo/Grey</material>
+    </gazebo>
+    <joint name="${prefix}razbot2_gripper_finger" type="prismatic">
+      <parent link="razbot2_arm_gripper_mounting_plate"/>
+      <child link="${prefix}razbot2_gripper_finger"/>
+      <axis xyz="0 0 0" rpy="0 0 0" />
+    </joint>
+   </xacro:macro>
 </robot>
